File: Kicad files/EnvOpenGamepad.kicad_sch (KiCad schematic)
At the start: 52 parts, among them J1 TYPE-C-31-M-12, J2 01x02 2.54mm pin header, SW1 B3SL-1025P, SW10 B3SL-1025P, SW11 EVQPU, SW12 EVQPUL, SW2 B3SL-1025P, SW3 B3SL-1025P, SW4 B3SL-1025P, SW5 B3SL-1025P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

Commit message: updated schematic and completed pcb wiring, generated pcb production files.
Connections:
- net BTN1: now also U2.9 (GPIO6)
- net BTN10: now also U2.2 (GPIO1)
- net BTN11: now also U2.6 (GPIO4)
- net BTN12: now also U2.7 (GPIO5)
- net BTN2: now also U2.10 (GPIO7)
- net BTN3: now also U2.11 (GPIO8)
- net BTN4: now also U2.12 (GPIO9)
- net BTN5: now also U2.27 (GPIO21)
- net BTN6: now also U2.26 (GPIO20)
- net BTN7: now also U2.25 (GPIO19)
- net BTN8: now also U2.24 (GPIO18)
- net BTN9: now also U2.1 (GPIO0)
Other:
- note added: "env"
