File: Kicad files/EnvOpenGamepad.kicad_pcb (KiCad board)
At the start: 2 copper layers, 100 x 75 mm, 52 parts, among them J1 TYPE-C-31-M-12, J2 01x02 2.54mm pin header, SW1 B3SL-1025P, SW10 B3SL-1025P, SW11 EVQPU, SW12 EVQPUL, SW2 B3SL-1025P, SW3 B3SL-1025P, SW4 B3SL-1025P, SW5 B3SL-1025P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

Commit message: updated schematic and completed pcb wiring, generated pcb production files.
Parts:
- moved H2 117.0 mm to (53.3, 60.6)
- moved H4 115.6 mm to (146.7, 129.4)
- moved C1 39.1 mm to (56.2, 114.8)
- moved C13 39.1 mm to (55.2, 114.8)
- moved C2 39.1 mm to (144.8, 114.2)
- moved C3 39.1 mm to (143.8, 114.2)
- moved R5 39.1 mm to (55.2, 123.0)
- moved R6 39.1 mm to (143.8, 123.3)
- moved R7 39.1 mm to (57.2, 114.8)
- moved R8 39.1 mm to (145.8, 114.2)
- moved U1 39.1 mm to (55.8, 119.0)
- moved U3 39.1 mm to (72.0, 119.0)
- moved U4 39.1 mm to (144.2, 119.0)
- moved U5 39.1 mm to (128.0, 119.0)
- moved SW6 28.3 mm to (134.6, 87.7)
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Connections:
- U2 pad 1: unconnected-(U2-GPIO0-Pad1) -> BTN9
- U2 pad 10: unconnected-(U2-GPIO7-Pad10) -> BTN2
- U2 pad 11: unconnected-(U2-GPIO8-Pad11) -> BTN3
- U2 pad 12: unconnected-(U2-GPIO9-Pad12) -> BTN4
- U2 pad 2: unconnected-(U2-GPIO1-Pad2) -> BTN10
- U2 pad 24: unconnected-(U2-GPIO18-Pad24) -> BTN8
- U2 pad 25: unconnected-(U2-GPIO19-Pad25) -> BTN7
- U2 pad 26: unconnected-(U2-GPIO20-Pad26) -> BTN6
- U2 pad 27: unconnected-(U2-GPIO21-Pad27) -> BTN5
- U2 pad 6: unconnected-(U2-GPIO4-Pad6) -> BTN11
- U2 pad 7: unconnected-(U2-GPIO5-Pad7) -> BTN12
- U2 pad 9: unconnected-(U2-GPIO6-Pad9) -> BTN1
Routing:
- net +3V3: track 13.4 -> 313.2 mm, vias 0 -> 9
- net I2C1_SDA: track 0.00 -> 179.2 mm, vias 0 -> 2
- net I2C1_SCL: track 0.00 -> 178.1 mm, vias 0 -> 3
- net BTN8: track 0.00 -> 85.3 mm
- net RT-ADC: track 0.00 -> 77.6 mm
- net LT-ADC: track 0.00 -> 76.1 mm
- net BTN12: track 0.00 -> 67.4 mm, vias 0 -> 3
- net BTN7: track 0.00 -> 63.1 mm
- net BTN2: track 0.00 -> 61.1 mm
- net Net-(U4-AIN0): track 0.00 -> 47.9 mm, vias 0 -> 1
- net BTN1: track 0.00 -> 47.1 mm
- net BTN11: track 0.00 -> 44.3 mm, vias 0 -> 1
- net BTN4: track 0.00 -> 43.9 mm
- net BTN5: track 0.00 -> 43.2 mm
- net BTN6: track 0.00 -> 39.7 mm
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Other:
- board size 100 x 75 mm -> 100 x 76 mm
- board text added: "EnvOpenGamePad"
- board text added: "POC-0.1"
- board text added: "env"

Commit message: unsure of current changes
Parts:
- moved H3 0.44 mm to (53.3, 129.4)
- moved H1 0.22 mm to (146.7, 60.6)
Changed lines of the file:
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@@
 		)
 		(fp_text user "3V3"
-			(at 12.9 -13.9 45)
+			(at 12.719188 -13.9 45)
 			(layer "F.SilkS")
 			(effects
@@
 		)
 		(fp_text user "GP21"
-			(at 13.054 8.9 45)
+			(at 13.042437 8.9 45)
 			(layer "F.SilkS")
 			(effects
@@
 		)
 		(fp_text user "3V3_EN"
-			(at 5.7 -15.6 45)
+			(at 13.486904 -17.2 45)
 			(layer "F.SilkS")
 			(effects
@@
 		)
 		(fp_text user "VBUS"
-			(at 13.3 -24.2 45)
+			(at 13.028968 -24.2 45)
 			(layer "F.SilkS")
 			(effects
@@
 		)
 		(fp_text user "GP17"
-			(at 13.054 21.59 45)
+			(at 13.042437 21.59 45)
 			(layer "F.SilkS")
 			(effects
@@
 		)
 		(fp_text user "GP26"
-			(at 13.054 -1.27 45)
+			(at 13.042437 -1.27 45)
 			(layer "F.SilkS")
 			(effects
@@
 		)
 		(fp_text user "GP18"
-			(at 13.054 16.51 45)
+			(at 13.042437 16.51 45)
 			(layer "F.SilkS")
 			(effects
@@
 		)
 		(fp_text user "GP27"
-			(at 13.054 -3.8 45)
+			(at 13.042437 -3.8 45)
 			(layer "F.SilkS")
 			(effects
@@
 		)
 		(fp_text user "VSYS"
-			(at 13.2 -21.59 45)
+			(at 12.961625 -21.59 45)
 			(layer "F.SilkS")
 			(effects
@@
 		)
 		(fp_text user "GP16"
-			(at 13.054 24.13 45)
+			(at 13.042437 24.13 45)
 			(layer "F.SilkS")
 			(effects
@@
 		)
 		(fp_text user "AGND"
-			(at 13.054 -6.35 45)
+			(at 13.042436 -6.35 45)
 			(layer "F.SilkS")
 			(effects
@@
 		)
 		(fp_text user "GP19"
-			(at 13.054 13.97 45)
+			(at 13.042437 13.97 45)
 			(layer "F.SilkS")
 			(effects
@@
 		)
 		(fp_text user "RUN"
-			(at 13 1.27 45)
+			(at 12.813469 1.27 45)
 			(layer "F.SilkS")
 			(effects
@@
 		)
 		(fp_text user "GP28"
-			(at 13.054 -9.144 45)
+			(at 13.042437 -9.144 45)
 			(layer "F.SilkS")
 			(effects
@@
 		)
 		(fp_text user "GP20"
-			(at 13.054 11.43 45)
+			(at 13.042437 11.43 45)
 			(layer "F.SilkS")
 			(effects
@@
 		)
 		(fp_text user "GP22"
-			(at 13.054 3.81 45)
+			(at 13.042437 3.81 45)
 			(layer "F.SilkS")
 			(effects
@@
 		)
 		(fp_text user "ADC_VREF"
-			(at 5.45 -9.85 45)
+			(at 13.985246 -12.6 45)
 			(layer "F.SilkS")
 			(effects
@@
 	(footprint "MountingHole:MountingHole_2.2mm_M2"
 		(layer "F.Cu")
-		(at 53.031306 129.045286)
+		(at 53.311822 129.379592)
 		(descr "Mounting Hole 2.2mm, no annular, M2")
 		(tags "mounting hole 2.2mm no annular m2")
@@
 	(footprint "MountingHole:MountingHole_2.2mm_M2"
 		(layer "F.Cu")
-		(at 146.535534 60.464466)
+		(at 146.688178 60.620408)
 		(descr "Mounting Hole 2.2mm, no annular, M2")
 		(tags "mounting hole 2.2mm no annular m2")
@@
 	)
 	(gr_line
-		(start 99.825501 121)
-		(end 124.825501 121)
-		(stroke
-			(width 0.2)
-			(type default)
-		)
-		(layer "F.SilkS")
-	)
-	(gr_line
-		(start 99.825501 121)
-		(end 74.8255 121)
-		(stroke
-			(width 0.2)
-			(type default)
-		)
-		(layer "F.SilkS")
-	)
-	(gr_line
 		(start 64 73)
 		(end 64 91)
@@
 	)
 	(gr_text "POC-0.1"
-		(at 100 94 0)
-		(layer "F.SilkS")
+		(at 100 59.3 -0)
+		(layer "B.SilkS")
 		(effects
 			(font
@@
 				(bold yes)
 			)
+			(justify mirror)
 		)
 	)
 	(gr_text "EnvOpenGamePad"
-		(at 100 92.5 0)
-		(layer "F.SilkS")
+		(at 100 57.8 -0)
+		(layer "B.SilkS")
 		(effects
 			(font
@@
 				(bold yes)
 			)
+			(justify mirror)
 		)
 	)
 	(gr_text "env"
-		(at 100 91.25 0)
+		(at 100 57.75 0)
 		(layer "F.SilkS")
 		(effects
@@
 			(polygon
 				(pts
-					(xy 98.85621 91.8725) (xy 98.781127 91.868385) (xy 98.704404 91.854355) (xy 98.633827 91.830368)
-					(xy 98.563915 91.794389) (xy 98.500906 91.749653) (xy 98.462735 91.714963) (xy 98.41216 91.656556)
-					(xy 98.370343 91.591246) (xy 98.34733 91.543871) (xy 98.321656 91.468222) (xy 98.308531 91.395348)
-					(xy 98.305199 91.333211) (xy 98.310177 91.258869) (xy 98.326964 91.181125) (xy 98.34733 91.125116)
-					(xy 98.383309 91.054981) (xy 98.428045 90.991851) (xy 98.462735 90.953658) (xy 98.521142 90.902756)
-					(xy 98.586452 90.86051) (xy 98.633827 90.837154) (xy 98.703018 90.812541) (xy 98.775586 90.798145)
-					(xy 98.844487 90.793923) (xy 98.918829 90.799075) (xy 98.996573 90.816446) (xy 99.052582 90.83752)
-					(xy 99.122717 90.874271) (xy 99.185847 90.919678) (xy 99.22404 90.954757) (xy 99.274942 91.013541)
-					(xy 99.317188 91.079435) (xy 99.340544 91.127315) (xy 99.365157 91.196541) (xy 99.379553 91.268711)
-					(xy 99.383775 91.336875) (xy 99.383775 91.450448) (xy 98.832763 91.450448) (xy 98.832763 91.262869)
-					(xy 99.202058 91.262869) (xy 99.186602 91.188681) (xy 99.174581 91.162486) (xy 99.132106 91.101234)
-					(xy 99.098377 91.069429) (xy 99.034444 91.027691) (xy 98.983705 91.005682) (xy 98.911752 90.986815)
-					(xy 98.844487 90.981502) (xy 98.771214 90.988279) (xy 98.70307 91.008613) (xy 98.635154 91.045836)
-					(xy 98.589864 91.084084) (xy 98.542542 91.143293) (xy 98.514392 91.196557) (xy 98.492953 91.267239)
-					(xy 98.486915 91.333211) (xy 98.49467 91.40944) (xy 98.514392 91.472063) (xy 98.551976 91.539155)
-					(xy 98.589864 91.583804) (xy 98.649305 91.630301) (xy 98.70307 91.65781) (xy 98.774145 91.678143)
-					(xy 98.850759 91.684895) (xy 98.85621 91.684921)
+					(xy 98.85621 58.3725) (xy 98.781127 58.368385) (xy 98.704404 58.354355) (xy 98.633827 58.330368)
+					(xy 98.563915 58.294389) (xy 98.500906 58.249653) (xy 98.462735 58.214963) (xy 98.41216 58.156556)
+					(xy 98.370343 58.091246) (xy 98.34733 58.043871) (xy 98.321656 57.968222) (xy 98.308531 57.895348)
+					(xy 98.305199 57.833211) (xy 98.310177 57.758869) (xy 98.326964 57.681125) (xy 98.34733 57.625116)
+					(xy 98.383309 57.554981) (xy 98.428045 57.491851) (xy 98.462735 57.453658) (xy 98.521142 57.402756)
+					(xy 98.586452 57.36051) (xy 98.633827 57.337154) (xy 98.703018 57.312541) (xy 98.775586 57.298145)
+					(xy 98.844487 57.293923) (xy 98.918829 57.299075) (xy 98.996573 57.316446) (xy 99.052582 57.33752)
+					(xy 99.122717 57.374271) (xy 99.185847 57.419678) (xy 99.22404 57.454757) (xy 99.274942 57.513541)
+					(xy 99.317188 57.579435) (xy 99.340544 57.627315) (xy 99.365157 57.696541) (xy 99.379553 57.768711)
+					(xy 99.383775 57.836875) (xy 99.383775 57.950448) (xy 98.832763 57.950448) (xy 98.832763 57.762869)
+					(xy 99.202058 57.762869) (xy 99.186602 57.688681) (xy 99.174581 57.662486) (xy 99.132106 57.601234)
+					(xy 99.098377 57.569429) (xy 99.034444 57.527691) (xy 98.983705 57.505682) (xy 98.911752 57.486815)
+					(xy 98.844487 57.481502) (xy 98.771214 57.488279) (xy 98.70307 57.508613) (xy 98.635154 57.545836)
+					(xy 98.589864 57.584084) (xy 98.542542 57.643293) (xy 98.514392 57.696557) (xy 98.492953 57.767239)
+					(xy 98.486915 57.833211) (xy 98.49467 57.90944) (xy 98.514392 57.972063) (xy 98.551976 58.039155)
+					(xy 98.589864 58.083804) (xy 98.649305 58.130301) (xy 98.70307 58.15781) (xy 98.774145 58.178143)
+					(xy 98.850759 58.184895) (xy 98.85621 58.184921)
 				)
 			)
 			(polygon
 				(pts
-					(xy 99.510537 91.352995) (xy 99.514723 91.278141) (xy 99.528997 91.201669) (xy 99.553402 91.131345)
-					(xy 99.590049 91.0609) (xy 99.635147 90.996843) (xy 99.669905 90.957688) (xy 99.728363 90.905515)
-					(xy 99.793828 90.862204) (xy 99.841364 90.838253) (xy 99.91072 90.813014) (xy 99.98328 90.798252)
-					(xy 100.052023 90.793923) (xy 100.127617 90.798988) (xy 100.199748 90.814183) (xy 100.262316 90.836788)
-					(xy 100.332607 90.873315) (xy 100.3962 90.918601) (xy 100.434874 90.953658) (xy 100.486446 91.012459)
-					(xy 100.529053 91.077855) (xy 100.552477 91.125116) (xy 100.578821 91.200215) (xy 100.592288 91.272586)
-					(xy 100.595708 91.33431) (xy 100.595708 91.8725) (xy 100.411793 91.8725) (xy 100.411793 91.336875)
-					(xy 100.403935 91.262076) (xy 100.383949 91.199855) (xy 100.348654 91.135608) (xy 100.307379 91.086648)
-					(xy 100.24723 91.038322) (xy 100.193074 91.009712) (xy 100.120604 90.9877) (xy 100.052023 90.981502)
-					(xy 99.979025 90.988737) (xy 99.910973 91.010444) (xy 99.845948 91.046597) (xy 99.796301 91.088114)
-					(xy 99.748091 91.148263) (xy 99.719731 91.202419) (xy 99.698291 91.277395) (xy 99.692254 91.352995)
+					(xy 99.510537 57.852995) (xy 99.514723 57.778141) (xy 99.528997 57.701669) (xy 99.553402 57.631345)
+					(xy 99.590049 57.5609) (xy 99.635147 57.496843) (xy 99.669905 57.457688) (xy 99.728363 57.405515)
+					(xy 99.793828 57.362204) (xy 99.841364 57.338253) (xy 99.91072 57.313014) (xy 99.98328 57.298252)
+					(xy 100.052023 57.293923) (xy 100.127617 57.298988) (xy 100.199748 57.314183) (xy 100.262316 57.336788)
+					(xy 100.332607 57.373315) (xy 100.3962 57.418601) (xy 100.434874 57.453658) (xy 100.486446 57.512459)
+					(xy 100.529053 57.577855) (xy 100.552477 57.625116) (xy 100.578821 57.700215) (xy 100.592288 57.772586)
+					(xy 100.595708 57.83431) (xy 100.595708 58.3725) (xy 100.411793 58.3725) (xy 100.411793 57.836875)
+					(xy 100.403935 57.762076) (xy 100.383949 57.699855) (xy 100.348654 57.635608) (xy 100.307379 57.586648)
+					(xy 100.24723 57.538322) (xy 100.193074 57.509712) (xy 100.120604 57.4877) (xy 100.052023 57.481502)
+					(xy 99.979025 57.488737) (xy 99.910973 57.510444) (xy 99.845948 57.546597) (xy 99.796301 57.588114)
+					(xy 99.748091 57.648263) (xy 99.719731 57.702419) (xy 99.698291 57.777395) (xy 99.692254 57.852995)
 				)
 			)
 			(polygon
 				(pts
-					(xy 101.362142 91.212677) (xy 101.569871 91.212677) (xy 101.252233 91.852716) (xy 101.252233 91.9117)
-					(xy 100.707083 90.793923) (xy 100.908217 90.793923) (xy 101.237944 91.495511) (xy 101.228785 91.492946)
+					(xy 101.362142 57.712677) (xy 101.569871 57.712677) (xy 101.252233 58.352716) (xy 101.252233 58.4117)
+					(xy 100.707083 57.293923) (xy 100.908217 57.293923) (xy 101.237944 57.995511) (xy 101.228785 57.992946)
 				)
 			)
